File: pcb/versie_2/versie_2/versie_2.kicad_pcb (KiCad board)
At the start: 2 copper layers, 32 x 61 mm, 3 parts, among them J2 Conn_01x04_Pin, J3 B4B-PH-SM4-TB__LF__SN_, U1 DFR0478

Commit message: PCB_update
Parts:
- J3: footprint Library:JST_B4B-PH-SM4-TB__LF__SN_ -> Library:CONN_B4B-ZR-SM4-TF_JST
- moved J3 0.86 mm to (201.9, 53.1)
Routing:
- net vcc: track 98.3 -> 122.5 mm
- net GND: track 81.4 -> 89.2 mm
- net TX_1: track 40.0 -> 41.6 mm
- net RX_1: track 43.4 -> 44.8 mm
Other:
- outline, holes or cut-outs redrawn

Commit message: PCB_update_finaal
Parts:
- J3: footprint Library:CONN_B4B-ZR-SM4-TF_JST -> Library:B4B-ZR
- moved J3 4.97 mm to (198.2, 56.4), turned to 0 degrees
