File: pcb/versie_2/versie_2/versie_2.kicad_sch (KiCad schematic)
At the start: 3 parts, among them J2 Conn_01x04_Pin, J3 B4B-PH-SM4-TB__LF__SN_, U1 DFR0654

Commit message: PCB_2eversie
Parts:
- removed U1: DFR0654, warre:MODULE_DFR0654, symbol warre:DFR0654
- added U1: DFR0478, Library:FIREBEETLE_ESP32, symbol footprints:DFR0478
- J2: footprint Connector_PinSocket_2.00mm:PinSocket_1x04_P2.00mm_Horizontal -> Library:GY-GPS6MV2
- J3: footprint Footprints:JST_B4B-PH-SM4-TB__LF__SN_ -> Library:JST_B4B-PH-SM4-TB__LF__SN_
Connections:
- net GND: now also U1.15 (GND)
- net RX: now also U1.34 (DI/IO16)
- net RX_1: now also U1.4 (IO26/D3)
- net TX: now also U1.35 (LRCK/IO17)
- net TX_1: now also U1.5 (IO27/D4)
- net vcc: now also U1.18 (VCC)
- no-connect marks 21 -> 32
Other:
- moved on the sheet: J2, J3

Commit message: PCB_update
Parts:
- J3: footprint Library:JST_B4B-PH-SM4-TB__LF__SN_ -> CONN_B4B-ZR-SM4-TF_JST; symbol B4B-PH-SM4-TB__LF__SN_:B4B-PH-SM4-TB__LF__SN_ -> footprints:B4B-ZR-SM4-TF_LFSN; Check_prices https://www.snapeda.com/parts/B4B-PH-SM4-TB%20(LF)(SN)/JST/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 -> https://www.snapeda.com/parts/B4B-ZR/JST/view-part/?ref=eda; Description_1 Socket; wire-board; male; PH; 2mm; PIN: 4; SMT; 100V; 2A; -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 -> Connector Header Surface Mount 4 position 0.059 (1.50mm); MF JST -> JST Sales; MP B4B-PH-SM4-TB (LF)(SN) -> B4B-ZR; Package NON STANDARD-4 JST -> None; SnapEDA_Link https://www.snapeda.com/parts/B4B-PH-SM4-TB%20(LF)(SN)/JST/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 -> https://www.snapeda.com/parts/B4B-ZR/JST/view-part/?ref=snap
Connections:
- net GND: no longer J3.SH1 (SHIELD), J3.SH2 (SHIELD)
- no-connect marks 32 -> 33

Commit message: PCB_update_finaal
Parts:
- J3: footprint CONN_B4B-ZR-SM4-TF_JST -> Library:B4B-ZR
Changed lines of the file:
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@@
 			)
 		)
-		(property "Footprint" "CONN_B4B-ZR-SM4-TF_JST"
+		(property "Footprint" "Library:B4B-ZR"
 			(at 124.46 100.33 0)
 			(effects

Commit message: pcb_update
Parts:
- added H1, H2, H3, H4, H5, H6, H7, H8: MountingHole_Pad, MountingHole:MountingHole_3.2mm_M3_ISO14580_Pad_TopBottom, symbol Mechanical:MountingHole_Pad
Connections:
- net GND: now also U1.MH1, U1.MH2, U1.MH3, U1.MH4, H1.1, H2.1, H3.1, H4.1, H5.1, H6.1, H7.1, H8.1
- no-connect marks 33 -> 29
Other:
- note added: "MountingHoles"
- moved on the sheet: J2, J3, U1
