File: pcb/versie_2/aiotp-project-NoxProject-versie2/aiotp-NoxProject.kicad_pcb (KiCad board)
At the start: 2 copper layers, 101 x 63.5 mm, 10 parts, among them J2 GPS connector, J3 Stemma connector, U1 DFR0478

Commit message: PCB en influx en node
Connections:
- U1 pad 31: unconnected-(U1-BCLK/IO14-Pad31) -> TX_1
- U1 pad 32: unconnected-(U1-MCLK/IO12-Pad32) -> RX_1
- U1 pad 4: RX_1 -> unconnected-(U1-IO26/D3-Pad4)
- U1 pad 5: TX_1 -> unconnected-(U1-IO27/D4-Pad5)
Routing:
- net RX_1: track 87.9 -> 117.2 mm
- net TX_1: track 101.5 -> 120.5 mm
Changed lines of the file:
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@@
 	(net 9 "unconnected-(U1-SCL{slash}IO22-Pad30)")
 	(net 10 "unconnected-(U1-IO8{slash}SD1-Pad13)")
-	(net 11 "unconnected-(U1-BCLK{slash}IO14-Pad31)")
+	(net 11 "unconnected-(U1-IO26{slash}D3-Pad4)")
 	(net 12 "unconnected-(U1-IO3{slash}RXD-Pad1)")
 	(net 13 "unconnected-(U1-IO13{slash}D7-Pad8)")
@@
 	(net 26 "unconnected-(U1-A1{slash}IO39-Pad20)")
 	(net 27 "unconnected-(U1-AREF-Pad16)")
-	(net 28 "unconnected-(U1-MCLK{slash}IO12-Pad32)")
+	(net 28 "unconnected-(U1-IO27{slash}D4-Pad5)")
 	(net 29 "unconnected-(U1-IO10{slash}D6-Pad7)")
 	(net 30 "unconnected-(U1-A2{slash}IO34-Pad21)")
@@
 		(property ki_fp_filters "CONN_B4B-ZR-SM4-TF_JST")
 		(sheetname "/")
-		(sheetfile "versie_2.kicad_sch")
+		(sheetfile "aiotp-NoxProject.kicad_sch")
 		(attr through_hole)
 		(fp_line
@@
 		(property ki_fp_filters "Pin* Test*")
 		(sheetname "/")
-		(sheetfile "versie_2.kicad_sch")
+		(sheetfile "aiotp-NoxProject.kicad_sch")
 		(attr exclude_from_pos_files)
 		(fp_circle
@@
 		(property ki_fp_filters "Pin* Test*")
 		(sheetname "/")
-		(sheetfile "versie_2.kicad_sch")
+		(sheetfile "aiotp-NoxProject.kicad_sch")
 		(attr exclude_from_pos_files)
 		(fp_circle
@@
 		(property ki_fp_filters "Connector*:*_1x??_*")
 		(sheetname "/")
-		(sheetfile "versie_2.kicad_sch")
+		(sheetfile "aiotp-NoxProject.kicad_sch")
 		(attr through_hole)
 		(fp_line
@@
 		(property ki_fp_filters "Pin* Test*")
 		(sheetname "/")
-		(sheetfile "versie_2.kicad_sch")
+		(sheetfile "aiotp-NoxProject.kicad_sch")
 		(attr exclude_from_pos_files)
 		(fp_circle
@@
 		(property ki_fp_filters "Pin* Test*")
 		(sheetname "/")
-		(sheetfile "versie_2.kicad_sch")
+		(sheetfile "aiotp-NoxProject.kicad_sch")
 		(attr exclude_from_pos_files)
 		(fp_circle
@@
 		(property ki_fp_filters "Pin* Test*")
 		(sheetname "/")
-		(sheetfile "versie_2.kicad_sch")
+		(sheetfile "aiotp-NoxProject.kicad_sch")
 		(attr exclude_from_pos_files)
 		(fp_circle
@@
 		)
 		(sheetname "/")
-		(sheetfile "versie_2.kicad_sch")
+		(sheetfile "aiotp-NoxProject.kicad_sch")
 		(attr through_hole)
 		(fp_line
@@
 			(layers "*.Cu" "*.Mask")
 			(remove_unused_layers no)
-			(net 6 "RX_1")
+			(net 11 "unconnected-(U1-IO26{slash}D3-Pad4)")
 			(pinfunction "IO26/D3")
-			(pintype "passive")
+			(pintype "passive+no_connect")
 		)
 		(pad "5" thru_hole circle
@@
 			(layers "*.Cu" "*.Mask")
 			(remove_unused_layers no)
-			(net 5 "TX_1")
+			(net 28 "unconnected-(U1-IO27{slash}D4-Pad5)")
 			(pinfunction "IO27/D4")
-			(pintype "passive")
+			(pintype "passive+no_connect")
 		)
 		(pad "6" thru_hole circle
@@
 			(layers "*.Cu" "*.Mask")
 			(remove_unused_layers no)
-			(net 11 "unconnected-(U1-BCLK{slash}IO14-Pad31)")
+			(net 5 "TX_1")
 			(pinfunction "BCLK/IO14")
-			(pintype "passive+no_connect")
+			(pintype "passive")
 		)
 		(pad "32" thru_hole circle
@@
 			(layers "*.Cu" "*.Mask")
 			(remove_unused_layers no)
-			(net 28 "unconnected-(U1-MCLK{slash}IO12-Pad32)")
+			(net 6 "RX_1")
 			(pinfunction "MCLK/IO12")
-			(pintype "passive+no_connect")
+			(pintype "passive")
 		)
 		(pad "33" thru_hole circle
@@
 		(property ki_fp_filters "Pin* Test*")
 		(sheetname "/")
-		(sheetfile "versie_2.kicad_sch")
+		(sheetfile "aiotp-NoxProject.kicad_sch")
 		(attr exclude_from_pos_files)
 		(fp_circle
@@
 	)
 	(segment
+		(start 158.348 126.448)
+		(end 155.9 124)
+		(width 0.2)
+		(layer "F.Cu")
+		(net 5)
+	)
+	(segment
+		(start 162.552 126.448)
+		(end 158.348 126.448)
+		(width 0.2)
+		(layer "F.Cu")
+		(net 5)
+	)
+	(segment
+		(start 127 93.8)
+		(end 105.16 93.8)
+		(width 0.2)
+		(layer "F.Cu")
+		(net 5)
+	)
+	(segment
+		(start 105.16 93.8)
+		(end 98.77 87.41)
+		(width 0.2)
+		(layer "F.Cu")
+		(net 5)
+	)
+	(segment
+		(start 155.9 124)
+		(end 155.9 122.7)
+		(width 0.2)
+		(layer "F.Cu")
+		(net 5)
+	)
+	(segment
 		(start 164 125)
-		(end 146.73 107.73)
+		(end 162.552 126.448)
 		(width 0.2)
 		(layer "F.Cu")
@@
 	)
 	(segment
-		(start 146.73 107.73)
-		(end 124.17 107.73)
+		(start 155.9 122.7)
+		(end 127 93.8)
 		(width 0.2)
 		(layer "F.Cu")
@@
 	)
 	(segment
-		(start 123.5 111.5)
-		(end 109.15675 97.15675)
+		(start 95.1 67.2)
+		(end 96.6 65.7)
 		(width 0.2)
 		(layer "B.Cu")
@@
 	)
 	(segment
-		(start 125.5 109.06)
-		(end 125.5 111)
+		(start 95.1 83.74)
+		(end 95.1 67.2)
 		(width 0.2)
 		(layer "B.Cu")
@@
 	)
 	(segment
-		(start 109.15675 97.15675)
+		(start 105.85675 65.7)
 		(end 109.15675 69)
 		(width 0.2)
@@
 	)
 	(segment
-		(start 125 111.5)
-		(end 123.5 111.5)
+		(start 98.77 87.41)
+		(end 95.1 83.74)
 		(width 0.2)
 		(layer "B.Cu")
@@
 	)
 	(segment
-		(start 124.17 107.73)
-		(end 125.5 109.06)
+		(start 96.6 65.7)
+		(end 105.85675 65.7)
 		(width 0.2)
 		(layer "B.Cu")
@@
 	)
 	(segment
-		(start 125.5 111)
-		(end 125 111.5)
+		(start 158.145574 91.795)
+		(end 157.396631 91.795)
 		(width 0.2)
-		(layer "B.Cu")
-		(net 5)
+		(layer "F.Cu")
+		(net 6)
 	)
 	(segment
 		(start 159.07 125)
-		(end 144.34 110.27)
+		(end 154.941 120.871)
 		(width 0.2)
 		(layer "F.Cu")
@@
 	)
 	(segment
-		(start 144.34 110.27)
-		(end 124.17 110.27)
+		(start 121.4 83.6)
+		(end 110.65675 72.85675)
 		(width 0.2)
 		(layer "F.Cu")
@@
 	)
 	(segment
-		(start 124.17 110.27)
-		(end 110.65675 96.75675)
+		(start 110.65675 72.85675)
+		(end 110.65675 69)
 		(width 0.2)
-		(layer "B.Cu")
+		(layer "F.Cu")
 		(net 6)
 	)
 	(segment
-		(start 110.65675 96.75675)
+		(start 157.396631 91.795)
+		(end 149.201631 83.6)
+		(width 0.2)
+		(layer "F.Cu")
+		(net 6)
+	)
+	(segment
+		(start 158.145574 96.252377)
+		(end 158.705 95.692951)
+		(width 0.2)
+		(layer "F.Cu")
+		(net 6)
+	)
+	(segment
+		(start 154.941 98.665803)
+		(end 157.354426 96.252377)
+		(width 0.2)
+		(layer "F.Cu")
+		(net 6)
+	)
+	(segment
+		(start 149.201631 83.6)
+		(end 121.4 83.6)
+		(width 0.2)
+		(layer "F.Cu")
+		(net 6)
+	)
+	(segment
+		(start 158.705 92.354426)
+		(end 158.145574 91.795)
+		(width 0.2)
+		(layer "F.Cu")
+		(net 6)
+	)
+	(segment
+		(start 154.941 120.871)
+		(end 154.941 98.665803)
+		(width 0.2)
+		(layer "F.Cu")
+		(net 6)
+	)
+	(segment
+		(start 158.705 95.692951)
+		(end 158.705 92.354426)
+		(width 0.2)
+		(layer "F.Cu")
+		(net 6)
+	)
+	(segment
+		(start 157.354426 96.252377)
+		(end 158.145574 96.252377)
+		(width 0.2)
+		(layer "F.Cu")
+		(net 6)
+	)
+	(segment
+		(start 110.65675 72.98325)
 		(end 110.65675 69)
 		(width 0.2)
 		(layer "B.Cu")
+		(net 6)
+	)
+	(segment
+		(start 98.77 84.87)
+		(end 110.65675 72.98325)
+		(width 0.2)
+		(layer "B.Cu")

Commit message: pcb
Parts:
- added A0_IN1: TestPoint, TestPoint:TestPoint_THTPad_D1.0mm_Drill0.5mm, F.Cu at (168.9, 125.0)
- added P1: Waveshare batterij connector, Library:JST_S2B-PH-SM4-TB, F.Cu at (183.2, 94.0)
- added R1: 100k, Resistor_SMD:R_0805_2012Metric, F.Cu at (177.7, 93.0)
- added R2: 270k, Resistor_SMD:R_0805_2012Metric, F.Cu at (177.7, 95.5)
- renumbered J2 to J1, J3 to J2
Connections:
- U1 pad 19: unconnected-(U1-A0/IO36-Pad19) -> A0_IN
Routing:
- net A0_IN: track 0.00 -> 109.4 mm
- net Batt+: track 0.00 -> 4.62 mm
